File: PCB/megadesk.kicad_sch (KiCad schematic)
At the start: 20 parts, among them J1 Interface, J2 FFC, J3 AVR-ISP-6, U1 L7812, U2 L7805, U3 ATtiny841-SS, U4 MCP2003B

Commit message: PCB revision v7
Parts:
- J2: footprint !Custom:FFC_10 -> megadesk:FB35-10N0-AHK
Connections:
- net B10: now reaches J2.10 (Pin_10)
- net B10: now also U3.10 (PA3)
- net B9: now reaches J2.9 (Pin_9)
- net B9: now also U3.13 (AREF/PA0)
- no-connect marks 11 -> 7

Commit message: change some footprints to new libraries, add ffc alternative
Parts:
- BZ1: footprint !Greg:Buzzer_Murata_PKMCS0909E4000-R1-HAND-SOLDER -> Buzzer_Beeper:Buzzer_Murata_PKMCS0909E
- D1, D2: footprint Diodes_SMD:D_SOD-323_HandSoldering -> Diode_SMD:D_SOD-323
- J1: footprint Pin_Headers:Pin_Header_Angled_1x03_Pitch2.54mm -> Connector_PinHeader_2.54mm:PinHeader_1x03_P2.54mm_Horizontal
- J2: footprint megadesk:FB35-10N0-AHK -> megadesk:F1004-H-10-20G-R; LCSC C508489 -> C668117
- J3: now left out of the parts list
- U4: footprint Housings_SOIC:SOIC-8 -> Package_SO:SOIC-8_3.9x4.9mm_P1.27mm
Changed lines of the file:
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@@
-(kicad_sch (version 20210621) (generator eeschema)
+(kicad_sch (version 20211123) (generator eeschema)
   (paper "USLetter")
-  (junction (at 92.71 59.69) (diameter 0) (color 0 0 0 0))
-  (junction (at 218.44 77.47) (diameter 0) (color 0 0 0 0))
-  (junction (at 45.72 35.56) (diameter 0) (color 0 0 0 0))
-  (junction (at 78.74 43.18) (diameter 0) (color 0 0 0 0))
-  (junction (at 198.12 69.85) (diameter 0) (color 0 0 0 0))
-  (junction (at 213.36 77.47) (diameter 0) (color 0 0 0 0))
-  (junction (at 78.74 35.56) (diameter 0) (color 0 0 0 0))
-  (junction (at 168.91 67.31) (diameter 0) (color 0 0 0 0))
-  (junction (at 45.72 43.18) (diameter 0) (color 0 0 0 0))
-  (junction (at 44.45 25.4) (diameter 0) (color 0 0 0 0))
-  (junction (at 19.05 35.56) (diameter 0) (color 0 0 0 0))
+  (junction (at 218.44 77.47) (diameter 0) (color 0 0 0 0)
+  )
+  (junction (at 78.74 43.18) (diameter 0) (color 0 0 0 0)
+  )
+  (junction (at 45.72 35.56) (diameter 0) (color 0 0 0 0)
+  )
+  (junction (at 92.71 59.69) (diameter 0) (color 0 0 0 0)
+  )
+  (junction (at 45.72 43.18) (diameter 0) (color 0 0 0 0)
+  )
+  (junction (at 213.36 77.47) (diameter 0) (color 0 0 0 0)
+  )
+  (junction (at 44.45 25.4) (diameter 0) (color 0 0 0 0)
+  )
+  (junction (at 19.05 35.56) (diameter 0) (color 0 0 0 0)
+  )
+  (junction (at 168.91 67.31) (diameter 0) (color 0 0 0 0)
+  )
+  (junction (at 198.12 69.85) (diameter 0) (color 0 0 0 0)
+  )
+  (junction (at 78.74 35.56) (diameter 0) (color 0 0 0 0)
+  )
   (no_connect (at 148.59 39.37))
   (no_connect (at 130.81 96.52))
@@
     (property "Reference" "J1" (id 0) (at 119.38 22.86 0))
     (property "Value" "Interface" (id 1) (at 119.38 33.02 0))
-    (property "Footprint" "Pin_Headers:Pin_Header_Angled_1x03_Pitch2.54mm" (id 2) (at 119.38 27.94 0)
+    (property "Footprint" "Connector_PinHeader_2.54mm:PinHeader_1x03_P2.54mm_Horizontal" (id 2) (at 119.38 27.94 0)
       (effects (font (size 1.27 1.27)) hide)
     )
@@
     (property "Reference" "D1" (id 0) (at 195.58 63.5 90))
     (property "Value" "1N4148" (id 1) (at 203.2 63.5 90))
-    (property "Footprint" "Diodes_SMD:D_SOD-323_HandSoldering" (id 2) (at 198.12 63.5 0)
+    (property "Footprint" "Diode_SMD:D_SOD-323" (id 2) (at 198.12 63.5 0)
       (effects (font (size 1.27 1.27)) hide)
     )
@@
     (property "Reference" "D2" (id 0) (at 212.09 67.31 0))
     (property "Value" "1N4148" (id 1) (at 212.09 72.39 0))
-    (property "Footprint" "Diodes_SMD:D_SOD-323_HandSoldering" (id 2) (at 212.09 69.85 0)
+    (property "Footprint" "Diode_SMD:D_SOD-323" (id 2) (at 212.09 69.85 0)
       (effects (font (size 1.27 1.27)) hide)
     )
@@
   )
   (symbol (lib_id "Device:C") (at 92.71 63.5 0) (unit 1)
-    (in_bom yes) (on_board yes)
+    (in_bom yes) (on_board no)
     (property "Reference" "C4" (id 0) (at 93.345 60.96 0)
       (effects (font (size 1.27 1.27)) (justify left))
@@
     (property "Reference" "J2" (id 0) (at 153.67 19.05 0))
     (property "Value" "FFC" (id 1) (at 153.67 46.99 0))
-    (property "Footprint" "megadesk:FB35-10N0-AHK" (id 2) (at 153.67 31.75 0)
+    (property "Footprint" "megadesk:F1004-H-10-20G-R" (id 2) (at 153.67 31.75 0)
       (effects (font (size 1.27 1.27)) hide)
     )
@@
       (effects (font (size 1.27 1.27)) hide)
     )
-    (property "LCSC" "C508489" (id 5) (at 153.67 31.75 0)
+    (property "LCSC" "C668117" (id 5) (at 153.67 31.75 0)
       (effects (font (size 1.27 1.27)) hide)
     )
@@
       (effects (font (size 1.27 1.27)) (justify left))
     )
-    (property "Footprint" "!Greg:Buzzer_Murata_PKMCS0909E4000-R1-HAND-SOLDER" (id 2) (at 150.495 86.36 90)
+    (property "Footprint" "Buzzer_Beeper:Buzzer_Murata_PKMCS0909E" (id 2) (at 150.495 86.36 90)
       (effects (font (size 1.27 1.27)) hide)
     )
@@
   )
   (symbol (lib_id "Connector:AVR-ISP-6") (at 63.5 83.82 0) (unit 1)
-    (in_bom yes) (on_board yes)
+    (in_bom no) (on_board yes)
     (property "Reference" "J3" (id 0) (at 55.1434 81.3816 0)
       (effects (font (size 1.27 1.27)) (justify right))
@@
     (property "Reference" "U4" (id 0) (at 182.88 63.5 0))
     (property "Value" "MCP2003B" (id 1) (at 182.88 66.04 0))
-    (property "Footprint" "Housings_SOIC:SOIC-8" (id 2) (at 182.88 86.36 0)
+    (property "Footprint" "Package_SO:SOIC-8_3.9x4.9mm_P1.27mm" (id 2) (at 182.88 86.36 0)
       (effects (font (size 1.27 1.27)) hide)
     )
@@
     )
     (path "/00000000-0000-0000-0000-00005aa5cdc1"
-      (reference "BZ1") (unit 1) (value "Buzzer") (footprint "!Greg:Buzzer_Murata_PKMCS0909E4000-R1-HAND-SOLDER")
+      (reference "BZ1") (unit 1) (value "Buzzer") (footprint "Buzzer_Beeper:Buzzer_Murata_PKMCS0909E")
     )
     (path "/00000000-0000-0000-0000-00005aa096b7"
@@
     )
     (path "/00000000-0000-0000-0000-00005aa07680"
-      (reference "D1") (unit 1) (value "1N4148") (footprint "Diodes_SMD:D_SOD-323_HandSoldering")
+      (reference "D1") (unit 1) (value "1N4148") (footprint "Diode_SMD:D_SOD-323")
     )
     (path "/00000000-0000-0000-0000-00005aa0777b"
-      (reference "D2") (unit 1) (value "1N4148") (footprint "Diodes_SMD:D_SOD-323_HandSoldering")
+      (reference "D2") (unit 1) (value "1N4148") (footprint "Diode_SMD:D_SOD-323")
     )
     (path "/00000000-0000-0000-0000-00005a83b312"
-      (reference "J1") (unit 1) (value "Interface") (footprint "Pin_Headers:Pin_Header_Angled_1x03_Pitch2.54mm")
+      (reference "J1") (unit 1) (value "Interface") (footprint "Connector_PinHeader_2.54mm:PinHeader_1x03_P2.54mm_Horizontal")
     )
     (path "/00000000-0000-0000-0000-00005aa53ce2"
-      (reference "J2") (unit 1) (value "FFC") (footprint "megadesk:FB35-10N0-AHK")
+      (reference "J2") (unit 1) (value "FFC") (footprint "megadesk:F1004-H-10-20G-R")
     )
     (path "/00000000-0000-0000-0000-00005dbf5698"
@@
     )
     (path "/cce9a479-26b7-42b5-a1ff-ecaef0005f68"
-      (reference "U4") (unit 1) (value "MCP2003B") (footprint "Housings_SOIC:SOIC-8")
-    )
-  )
+      (reference "U4") (unit 1) (value "MCP2003B") (footprint "Package_SO:SOIC-8_3.9x4.9mm_P1.27mm")
+    )
+  )

Commit message: pcb revision only
Parts:
- added TP1, TP2: TestPoint, TestPoint:TestPoint_Pad_D1.5mm, symbol Connector:TestPoint
- added TP3: TPDN, TestPoint:TestPoint_Pad_D1.5mm, symbol Connector:TestPoint
- added TP4: TPUP, TestPoint:TestPoint_Pad_D1.5mm, symbol Connector:TestPoint
- BZ1: LCSC C255319 -> C391035
- U1: LCSC C67851 -> C16424; Notes 35V INPUT -> C16424; Part Number MC78M12CDTRKGOSTR -> 7812
- U2: LCSC C58069 -> C55509; Part Number MC78M05CDTRKGOSTR -> 7805
Connections:
- net Bdown: now also TP3.1
- net Bup: now also TP4.1
- new net: TP1.1, TP2.1

Commit message: Update to 1624 (v9)
Parts:
- removed U3: ATtiny841-SS, Package_SO:SOIC-14_3.9x8.7mm_P1.27mm, symbol MCU_Microchip_ATtiny:ATtiny841-SS
- added U3: ATtiny1624-SS, Package_SO:SOIC-14_3.9x8.7mm_P1.27mm, symbol MCU_Microchip_ATtiny:ATtiny1624-SS
Connections:
- net RST is gone; now on net GND: J3.5 (~{RST})
- net +5V: now also U3.1 (VCC)
- net B10: now also U3.13 (PA3)
- net B9: now also U3.2 (PA4)
- net Bdown: now also U3.4 (PA6)
- net Bup: now also U3.3 (PA5)
- net GND: now also U3.14 (GND)
- net RXD1: now reaches R3.2, U4.1 (RXD)
- net RXD1: now also U3.12 (PA2)
- net BEEP: now reaches BZ1.1 (-)
- net BEEP: now also U3.5 (PA7)
- net TXD1: now reaches U4.4 (TXD)
- net TXD1: now also U3.11 (PA1)
- net MISO renamed UPDI
- net UPDI: now also U3.10 (~{RESET}/PA0)
- net MOSI renamed TXD0
- net TXD0: now also U3.7 (PB2)
- net SCK renamed RXD0
- net RXD0: now also U3.6 (PB3)
- no-connect marks 7 -> 8
Other:
- note removed: "Optional beeper"
- moved on the sheet: C4
