File: PCB/megadesk.kicad_sch (KiCad schematic)
At the start: 24 parts, among them J1 Interface, J2 FFC, J3 AVR-ISP-6, U1 L7812, U2 L7805, U3 ATtiny1624-SS, U4 MCP2003B

Commit message: esp32c3mini
Parts:
- removed C4: DNP, Capacitor_SMD:C_0805_2012Metric, symbol Device:C
- removed C5: 0.1uF, Capacitor_SMD:C_0805_2012Metric, symbol Device:C
- removed J3: AVR-ISP-6, Connector_PinHeader_2.54mm:PinHeader_2x03_P2.54mm_Vertical, symbol Connector:AVR-ISP-6
- removed TP1, TP2: TestPoint, TestPoint:TestPoint_Pad_D1.5mm, symbol Connector:TestPoint
- removed TP3: TPDN, TestPoint:TestPoint_Pad_D1.5mm, symbol Connector:TestPoint
- removed TP4: TPUP, TestPoint:TestPoint_Pad_D1.5mm, symbol Connector:TestPoint
- removed U2: L7805, Package_TO_SOT_SMD:TO-252-3_TabPin2, symbol Regulator_Linear:L7805
- removed U3: ATtiny1624-SS, Package_SO:SOIC-14_3.9x8.7mm_P1.27mm, symbol MCU_Microchip_ATtiny:ATtiny1624-SS
- added C10: 10uF (50V), Capacitor_SMD:C_1206_3216Metric, symbol Device:C_Small
- added C4: 10uF, Capacitor_SMD:C_0603_1608Metric, symbol Device:C_Small
- added C7: 4.7uF (50V), Capacitor_SMD:C_1206_3216Metric, symbol Device:C_Small
- added C8: 0.1uF (50V), Capacitor_SMD:C_0402_1005Metric, symbol Device:C_Small
- added C9: 33pF, Capacitor_SMD:C_0402_1005Metric, symbol Device:C_Small
- added D4: 40V/1A, Diode_SMD:D_SOD-123, symbol Device:D_Schottky
- added J3: eflashy32, Connector_PinHeader_2.54mm:PinHeader_1x06_P2.54mm_Vertical, symbol Connector_Generic:Conn_01x06
- added L2: 2.2uH (50mA), Inductor_SMD:L_0805_2012Metric, symbol Device:L
- added R10: 124k, Resistor_SMD:R_0805_2012Metric, symbol Device:R_Small
- added R2: 10k, Resistor_SMD:R_0402_1005Metric, symbol Device:R_Small
- added R8: 1k, Resistor_SMD:R_0402_1005Metric, symbol Device:R
- added R9: 40.2k, Resistor_SMD:R_0603_1608Metric, symbol Device:R_Small
- added U2: ESP32-C3-MINI-1, !megadeskcompanion:ESP32-C3-MINI-1, symbol RF_Module:ESP32-C3-MINI-1
- added U3: BL9342, Package_TO_SOT_SMD:SOT-23-6, symbol !megadesk:BL9342
- BZ1: LCSC C391035 -> C255319
- C3: footprint Capacitor_SMD:C_0805_2012Metric -> Capacitor_SMD:C_0402_1005Metric; LCSC C49678 -> C1525
- J1: LCSC C376121 -> DNP
- J2: footprint megadesk:F1004-H-10-20G-R -> Connector_FFC-FPC:TE_1-84953-0_1x10-1MP_P1.0mm_Horizontal; LCSC C668117 -> C481254
- R1, R6: footprint Resistor_SMD:R_0603_1608Metric -> Resistor_SMD:R_0402_1005Metric; LCSC C21190 -> C11702
- R3, R4, R5: footprint Resistor_SMD:R_0603_1608Metric -> Resistor_SMD:R_0402_1005Metric; LCSC C23162 -> C25900
- U1: footprint Package_TO_SOT_SMD:TO-252-3_TabPin2 -> Package_TO_SOT_SMD:SOT-89-3; LCSC C16424 -> C347272; Notes C16424 -> 35V INPUT; Part Number 7812 -> UMW78L12
- U4: LCSC (none) -> C152207
Connections:
- net +12V: now also U1.1 (OUT); no longer U1.3 (OUT)
- net +24V: now also U1.3 (IN), C7.2, R8.1, U3.5 (VIN); no longer U1.1 (IN)
- net B10: now also U2.19 (IO5)
- net B9: now also U2.13 (IO1)
- net Bdown: now also U2.18 (IO4)
- net Bup: now also U2.6 (IO3)
- net GND: now also C10.2, C4.1, C7.1, D4.2 (A), J3.1 (Pin_1), R9.1, U2.1 (GND), U2.11 (GND), U2.14 (GND), U2.2 (GND), U2.36 (GND), U2.37 (GND), U2.38 (GND), U2.39 (GND), U2.40 (GND), U2.41 (GND), U2.42 (GND), U2.43 (GND), U2.44 (GND), U2.45 (GND), U2.46 (GND), U2.47 (GND), U2.48 (GND), U2.49 (GND), U2.50 (GND), U2.51 (GND), U2.52 (GND), U2.53 (GND), U3.2 (GND)
- net +5V renamed +3V3
- net +3V3: now also C10.1, C4.2, C9.2, J3.4 (Pin_4), L2.2, R10.2, R2.1, U2.3 (VDD)
- net BEEP: no longer names the net of BZ1.1 (-)
- net BEEP: now also U2.21 (IO7)
- net RXD1 renamed RXD
- net RXD: now also J3.3 (Pin_3), U2.30 (IO20/RXD)
- net TXD1 renamed TXD
- net TXD: now also J3.2 (Pin_2), U2.31 (IO21/TXD)
- new net: C8.2, D4.1 (K), L2.1, U3.6 (SW)
- new net: C9.1, R10.1, R9.2, U3.3 (FB)
- new net: R8.2, U3.4 (EN)
- new net: C8.1, U3.1 (BOOT)
- new net EN: J3.5 (Pin_5), R2.2, U2.8 (EN)
- new net GPIO0: J3.6 (Pin_6), U2.23 (IO9)
Other:
- note added: "12V Regulation"
- note added: "12V consumption by LIN bus typically 2-3mA"
- note added: "Bootstrap 2,8,9"
- note added: "C3 uses GPIO9 now"
- note added: "Output(TX) from eflashy32"
- note added: "Programming"
- note removed: "Power Regulation"
- note removed: "Volume control"
- moved on the sheet: BZ1, C1, C3, J1, J2, R5, U1

Commit message: esp rev2
Parts:
- removed U1: L7812, Package_TO_SOT_SMD:SOT-89-3, symbol Regulator_Linear:L7812
- removed U4: MCP2003B, Package_SO:SOIC-8_3.9x4.9mm_P1.27mm, symbol megadesk:MCP2003B
- added R11, R7: 10k, Resistor_SMD:R_0402_1005Metric, symbol Device:R_Small
- added TP1: RXD, TestPoint:TestPoint_Pad_D2.0mm, symbol Connector:TestPoint
- added TP2: TXD, TestPoint:TestPoint_Pad_D2.0mm, symbol Connector:TestPoint
- added TP3: GND, TestPoint:TestPoint_Pad_D2.0mm, symbol Connector:TestPoint
- added TP4: 3V3, TestPoint:TestPoint_Pad_D2.0mm, symbol Connector:TestPoint
- added U1: L78L12_SOT89, Package_TO_SOT_SMD:SOT-89-3, symbol Regulator_Linear:L78L12_SOT89
- added U4: MCP2003B, Package_SO:SOIC-8_3.9x4.9mm_P1.27mm, symbol !megadesk:MCP2003B
- L2: value 2.2uH (50mA) -> 2.2uH; footprint Inductor_SMD:L_0805_2012Metric -> megadesk:L_Sunlord_SWPA3015S; LCSC C1043 -> C43389; PN CMI201209U2R2KT -> SWPA3015S2R2NT
- R10: footprint Resistor_SMD:R_0805_2012Metric -> Resistor_SMD:R_0402_1005Metric; LCSC C204195 -> C36777
- U2: footprint !megadeskcompanion:ESP32-C3-MINI-1 -> Espressif:ESP32-C3-MINI-1
- U3: value BL9342 -> BL9342 / MP2451
Connections:
- net +12V: now also U1.1 (OUT)
- net +24V: now also R8.2, U3.4 (EN), U1.3 (IN)
- net +3V3: now also R11.1, R7.1, TP4.1
- net GND: now also TP3.1, U1.2 (GND), U4.5 (VSS)
- net LINBUS: now also U4.6 (LBUS)
- net RXD: now also TP1.1, U4.1 (RXD)
- net TXD: now also TP2.1, U4.4 (TXD)
- net at R5.1: now also U4.3 (WAKE)
- net at R4.1: now also U4.2 (CS)
- net at D1.1 (K), D2.2 (A): now also U4.7 (VBB)
- net SW: now reaches C8.2, D4.1 (K), L2.1, U3.6 (SW)
- net at U2.22 (IO8): now also R11.2
- net at U2.5 (IO2): now also R7.2
- net FB: now reaches C9.1, R10.1, R9.2, U3.3 (FB)
- net BOOT: now reaches C8.1, U3.1 (BOOT)
- no-connect marks 8 -> 11

Commit message: ugh v3
Connections:
- net RXD: now also U2.27 (IO19/D+); no longer J3.3 (Pin_3), TP1.1, U2.30 (IO20/RXD)
- net TXD: now also U2.26 (IO18/D-); no longer J3.2 (Pin_2), TP2.1, U2.31 (IO21/TXD)
- new net PROGRXD: J3.3 (Pin_3), TP1.1, U2.30 (IO20/RXD)
- new net PROGTXD: J3.2 (Pin_2), TP2.1, U2.31 (IO21/TXD)
- no-connect marks 11 -> 9
Changed lines of the file:
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@@
   (no_connect (at 139.7 24.13))
   (no_connect (at 78.74 81.28))
-  (no_connect (at 78.74 109.22))
   (no_connect (at 78.74 96.52))
   (no_connect (at 78.74 106.68))
-  (no_connect (at 78.74 111.76))
   (no_connect (at 139.7 26.67))
   (no_connect (at 139.7 29.21))
@@
     (stroke (width 0) (type default) (color 0 0 0 0))
   )
+  (wire (pts (xy 78.74 111.76) (xy 81.28 111.76))
+    (stroke (width 0) (type default) (color 0 0 0 0))
+  )
   (wire (pts (xy 170.18 133.35) (xy 170.18 135.89))
     (stroke (width 0) (type default) (color 0 0 0 0))
@@
   (wire (pts (xy 213.36 77.47) (xy 218.44 77.47))
     (stroke (width 0) (type solid) (color 0 0 0 0))
+  )
+  (wire (pts (xy 78.74 109.22) (xy 81.28 109.22))
+    (stroke (width 0) (type default) (color 0 0 0 0))
   )
   (wire (pts (xy 168.91 67.31) (xy 172.72 67.31))
@@
     (effects (font (size 1 1)) (justify left bottom))
   )
-  (text "Output(TX) from eflashy32" (at 80.01 35.56 0)
+  (text "Output(TX) from eflashy32" (at 46.99 35.56 0)
     (effects (font (size 1 1)) (justify left bottom))
   )
@@
     (effects (font (size 1.27 1.27)) (justify right bottom))
   )
-  (label "RXD" (at 81.28 116.84 0)
+  (label "RXD" (at 81.28 111.76 0)
+    (effects (font (size 1.27 1.27)) (justify left bottom))
+  )
+  (label "PROGTXD" (at 76.2 38.1 0)
     (effects (font (size 1.27 1.27)) (justify left bottom))
   )
@@
     (effects (font (size 1.27 1.27)) (justify left bottom))
   )
+  (label "PROGTXD" (at 78.105 61.595 180)
+    (effects (font (size 1.27 1.27)) (justify right bottom))
+  )
+  (label "PROGRXD" (at 81.28 116.84 0)
+    (effects (font (size 1.27 1.27)) (justify left bottom))
+  )
   (label "EN" (at 41.91 81.28 0)
     (effects (font (size 1.27 1.27)) (justify left bottom))
   )
-  (label "TXD" (at 81.28 114.3 0)
+  (label "TXD" (at 81.28 109.22 0)
     (effects (font (size 1.27 1.27)) (justify left bottom))
   )
@@
     (effects (font (size 1.524 1.524)) (justify left bottom))
   )
-  (label "TXD" (at 78.105 61.595 180)
-    (effects (font (size 1.27 1.27)) (justify right bottom))
-  )
   (label "SW" (at 170.18 138.43 0)
     (effects (font (size 1.524 1.524)) (justify left bottom))
   )
-  (label "RXD" (at 76.2 35.56 0)
-    (effects (font (size 1.27 1.27)) (justify left bottom))
-  )
-  (label "TXD" (at 76.2 38.1 0)
-    (effects (font (size 1.27 1.27)) (justify left bottom))
-  )
-  (label "RXD" (at 78.105 59.055 180)
+  (label "PROGRXD" (at 78.105 59.055 180)
     (effects (font (size 1.27 1.27)) (justify right bottom))
   )
+  (label "PROGTXD" (at 81.28 114.3 0)
+    (effects (font (size 1.27 1.27)) (justify left bottom))
+  )
+  (label "PROGRXD" (at 76.2 35.56 0)
+    (effects (font (size 1.27 1.27)) (justify left bottom))
+  )
   (label "EN" (at 76.2 30.48 0)

Commit message: pipelines
Parts:
- added C?: 1uF, symbol Device:C_Small
Connections:
- net EN: now also C?.1
- net GND: now also C?.2
Changed lines of the file:
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@@
   (junction (at 218.44 77.47) (diameter 0) (color 0 0 0 0)
+  )
+  (junction (at 35.56 81.28) (diameter 0) (color 0 0 0 0)
   )
   (junction (at 200.025 138.43) (diameter 0) (color 0 0 0 0)
@@
   )
   (wire (pts (xy 78.74 91.44) (xy 82.55 91.44))
+    (stroke (width 0) (type default) (color 0 0 0 0))
+  )
+  (wire (pts (xy 35.56 81.28) (xy 35.56 83.82))
     (stroke (width 0) (type default) (color 0 0 0 0))
   )
@@
     (pin "1")
   )
+  (symbol (lib_id "power:GND") (at 35.56 88.9 0) (unit 1)
+    (in_bom yes) (on_board yes)
+    (property "Reference" "#PWR?" (id 0) (at 35.56 95.25 0)
+      (effects (font (size 1.27 1.27)) hide)
+    )
+    (property "Value" "GND" (id 1) (at 35.56 92.71 0))
+    (property "Footprint" "" (id 2) (at 35.56 88.9 0)
+      (effects (font (size 1 1)) hide)
+    )
+    (property "Datasheet" "" (id 3) (at 35.56 88.9 0)
+      (effects (font (size 1 1)) hide)
+    )
+    (pin "1")
+  )
   (symbol (lib_id "!megadesk:MCP2003B") (at 182.88 74.93 0) (unit 1)
     (in_bom yes) (on_board yes) (fields_autoplaced)
@@
     (pin "1")
   )
+  (symbol (lib_id "Device:C_Small") (at 35.56 86.36 0) (unit 1)
+    (in_bom yes) (on_board yes) (fields_autoplaced)
+    (property "Reference" "C?" (id 0) (at 38.1 85.0962 0)
+      (effects (font (size 1.27 1.27)) (justify left))
+    )
+    (property "Value" "1uF" (id 1) (at 38.1 87.6362 0)
+      (effects (font (size 1.27 1.27)) (justify left))
+    )
+    (property "Footprint" "" (id 2) (at 35.56 86.36 0)
+      (effects (font (size 1.27 1.27)) hide)
+    )
+    (property "Datasheet" "~" (id 3) (at 35.56 86.36 0)
+      (effects (font (size 1.27 1.27)) hide)
+    )
+    (pin "1")
+    (pin "2")
+  )
   (symbol (lib_id "Device:R") (at 143.51 137.16 0) (unit 1)
     (in_bom yes) (on_board yes)
@@
       (reference "#PWR0114") (unit 1) (value "GND") (footprint "")
     )
+    (path "/37546594-f12c-4685-b2c4-beac38e27721"
+      (reference "#PWR?") (unit 1) (value "GND") (footprint "")
+    )
     (path "/00000000-0000-0000-0000-00005aa5cdc1"
       (reference "BZ1") (unit 1) (value "Buzzer") (footprint "Buzzer_Beeper:Buzzer_Murata_PKMCS0909E")
@@
       (reference "C10") (unit 1) (value "10uF (50V)") (footprint "Capacitor_SMD:C_1206_3216Metric")
     )
+    (path "/75b970ec-ca1c-4e51-8f39-fa282882b59c"
+      (reference "C?") (unit 1) (value "1uF") (footprint "")
+    )
     (path "/00000000-0000-0000-0000-00005aa07680"
