File: pcb/megadesk.kicad_sch (KiCad schematic)
At the start: 27 parts, among them J2 FFC, J3 AVR-ISP-6, J4 Interface, U1 7812, U2 HT7550-1, U3 ATtiny841-SS, U4 MCP2003B

Commit message: silkscreen change
Connections:
- net AVRTX: now reaches J4.5 (Pin_5), R7.2
- net AVRRX: now reaches J4.4 (Pin_4), R2.2
Other:
- moved on the sheet: BZ1, R1, R2, R7

Commit message: decoupling
Parts:
- added D3: SMF33A, Diode_SMD:D_SOD-123F, symbol Device:D_Schottky
- C4: value DNP -> 0.1uF; LCSC (none) -> C49678; now fitted
Connections:
- net +24V: now also D3.1 (K)
- net GND: now also D3.2 (A)
Other:
- moved on the sheet: C2, C3, C5, U1, U2
